Commit message: cognitive_architecture_update_1

File: src/robot/robot.urdf (robot description, URDF)
Before this commit: robot mobile_manipulator, 18 links, 17 joints
Links:
- added link lidar_link, mass 0.2; collision cylinder length=0.02 radius=0.03; visual box size=0.6 0.01 0.01
Joints:
- added joint lidar_joint: type fixed, parent base_link, child lidar_link, origin xyz=0.31 0 0.16 rpy=0 0 0
- joint camera_joint: origin xyz=0.04 0 0 rpy=0 1.5708 0 -> xyz=0.04 0 0 rpy=0 -1.5708 0

Commit message: cognitive_architecture_update_2

File: src/robot/robot.urdf (robot description, URDF)
Before this commit: robot mobile_manipulator, 19 links, 18 joints
Links:
- link lidar_link: mass 0.2 -> 0.25; geometry collision box size=0.05 0.05 0.04; visual box size=0.05 0.05 0.04
